File: hardware/esp-sensor/IDM-RoomSensor-ESP-B-ES2-C6.kicad_sch (KiCad schematic)
At the start: 67 parts, among them J1 1-2834011-4 / IDM 43 TEMP / 4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, J2 1-2834011-4 / RS485 A / B / C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, J3 TYPE-C-31-M-12, J4 EXPANSION, SW1 RESET, SW2 BOOT, U1 LMR36510ADDAR 24V-to-5V, U2 AP2112K-3.3TRG1, U3 ESP32-C6-WROOM-1-N16 (pins pe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, U4 SHT45-AD1B-R2, U5 MCP4725A0T-E/CH, U6 OPA197IDBVR, U7 ADM2587EBRWZ

Commit message: fix(hardware): correct C6 JLCPCB part mappings
Parts:
- R9: value 21k 0.1% -> 21k 1% CAL
Changed lines of the file:
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@@
       (effects (font (size 1.27 1.27)))
     )
-    (property "Value" "21k 0.1%" (at 270.51 69.85000000000001 0)
+    (property "Value" "21k 1% CAL" (at 270.51 69.85000000000001 0)
       (effects (font (size 1.27 1.27)))
     )

Commit message: fix(hardware): reduce isolated RS485 assembly cost
Parts:
- removed C15: 10n, Capacitor_SMD:C_0805_2012Metric, symbol Device:C
- removed FB1: 600R@100MHz ferrite, Inductor_SMD:L_0805_2012Metric, symbol Device:L
- removed U7: ADM2587EBRWZ, Package_SO:SOIC-20W_7.5x12.8mm_P1.27mm, symbol Interface_UART:ADM2587E
- added U7: CA-IS3092W, Package_SO:SOIC-16W_7.5x10.3mm_P1.27mm, symbol Connector_Generic:Conn_02x08_Odd_Even
Connections:
- net +3V3: now also U7.1 (Pin_1)
- net GND: now also U7.2 (Pin_2), U7.8 (Pin_8)
- net RS485_A: now also U7.12 (Pin_12)
- net RS485_B: now also U7.13 (Pin_13)
- net RS485_COM: now also U7.10 (Pin_10), U7.15 (Pin_15), U7.9 (Pin_9)
- net RS485_DE: now also U7.4 (Pin_4), U7.5 (Pin_5)
- net RS485_RX: now also U7.3 (Pin_3)
- net RS485_TX: now also U7.6 (Pin_6)
- net VISO: now also U7.16 (Pin_16)
- no-connect marks 16 -> 19
