File: hardware/esp-sensor/IDM-RoomSensor-ESP-B-ES4-AIR-R2.kicad_pcb (KiCad board)
At the start: 4 copper layers, 130 x 100 mm, 119 parts, among them J1 MX205R PUSH-IN 43/42/41/40, J2 MX205R PUSH-IN RS485 A/B/COM/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, J3 USB-C, J4 EXPANSION, J5 1WIRE A 3V/DQ/GND, J6 1WIRE B 3V/DQ/GND, J7 CONTACT 1/COM/2, J8 0-10V IN/GND, J9 RELAY COM/NO/NC, K1 HFD4/5, Q1 2N7002 VIN LED, Q2 2N7002 RELAY, SW1 RESET, SW2 BOOT, SW3 TERM ON/OFF, SW4 SERVICE, U1 LMR36510ADDAR, U10 BMP390, U11 AP2112K-3.3 AIR, U2 AP2112K-3.3, U3 ESP32-C6-WROOM-1-N16, U4 SHT45, U5 MCP4725A0T, U6 OPA197IDBVR, U7 CA-IS3092W, U8 SCD41-D-R1, U9 SGP41-D-R4

Commit message: Use stocked ESP32-C6 N8 and BMP388 for B-ES4 R2
Parts:
- U10: value BMP390 -> BMP388
- U3: value ESP32-C6-WROOM-1-N16 -> ESP32-C6-WROOM-1-N8
Other:
- board text added: "SGP41 VOC/NOx | BMP388 hPa"
- board text removed: "SGP41 VOC/NOx | BMP390 hPa"
Changed lines of the file:
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@@
 			)
 		)
-		(property "Value" "ESP32-C6-WROOM-1-N16"
+		(property "Value" "ESP32-C6-WROOM-1-N8"
 			(at 0 0 0)
 			(layer "F.Fab")
@@
 			)
 		)
-		(property "Value" "BMP390"
+		(property "Value" "BMP388"
 			(at 0 4.78 0)
 			(layer "F.Fab")
@@
 			)
 		)
-		(property "LCSC Part" "C5124834"
+		(property "LCSC Part" "C779278"
 			(at 0 0 0)
 			(layer "F.Fab")
@@
 		)
 	)
-	(gr_text "SGP41 VOC/NOx | BMP390 hPa"
+	(gr_text "SGP41 VOC/NOx | BMP388 hPa"
 		(at 44 106.8 0)
 		(layer "F.SilkS")
